File: board/Schematic/rough.sch (EAGLE design)
At the start: 12 parts

Commit message: added circuit protection
Parts:
- added F1, F2: 10AMP, fuse:SH22,5
Connections:
- new net N$7: D3.A, F2.1
- net N$2: now also F1.2
Other:
- moved on the sheet: C1, D3
Changed lines of the file:
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@@
 <part name="U$1" library="Test" deviceset="LT3652" device=""/>
 <part name="SUPPLY2" library="supply2" deviceset="GND" device=""/>
-<part name="SUPPLY5" library="supply2" deviceset="GND" device=""/>
-<part name="SUPPLY6" library="supply2" deviceset="GND" device=""/>
 <part name="SUPPLY7" library="supply2" deviceset="GND" device=""/>
 <part name="R1" library="resistor" deviceset="R-US_" device="R1206" value="0.05"/>
@@
 <part name="R2" library="rcl" deviceset="R-US_" device="M2012" value="634K"/>
 <part name="R3" library="rcl" deviceset="R-US_" device="M2012" value="412K"/>
+<part name="F1" library="fuse" deviceset="SH22,5" device="" value="10AMP"/>
+<part name="F2" library="fuse" deviceset="SH22,5" device="" value="10AMP"/>
 </parts>
 <sheets>
@@
 </plain>
 <instances>
-<instance part="SUPPLY1" gate="GND" x="12.7" y="73.66"/>
+<instance part="SUPPLY1" gate="GND" x="25.4" y="73.66"/>
 <instance part="SUPPLY3" gate="GND" x="76.2" y="25.4"/>
 <instance part="SUPPLY4" gate="GND" x="35.56" y="45.72"/>
-<instance part="C1" gate="G$1" x="12.7" y="83.82"/>
+<instance part="C1" gate="G$1" x="25.4" y="83.82"/>
 <instance part="C2" gate="G$1" x="86.36" y="48.26" rot="R180"/>
 <instance part="C3" gate="G$1" x="78.74" y="71.12"/>
 <instance part="INDUCTOR" gate="G$1" x="93.98" y="71.12" rot="R90"/>
 <instance part="U$1" gate="G$2" x="53.34" y="55.88" rot="R270"/>
-<instance part="SUPPLY2" gate="GND" x="53.34" y="33.02"/>
-<instance part="SUPPLY5" gate="GND" x="53.34" y="25.4"/>
-<instance part="SUPPLY6" gate="GND" x="45.72" y="25.4"/>
+<instance part="SUPPLY2" gate="GND" x="53.34" y="35.56"/>
 <instance part="SUPPLY7" gate="GND" x="86.36" y="43.18"/>
 <instance part="R1" gate="G$1" x="88.9" y="58.42"/>
@@
 <instance part="SUPPLY8" gate="GND" x="60.96" y="78.74"/>
 <instance part="D1" gate="G$1" x="76.2" y="58.42" rot="R90"/>
-<instance part="D3" gate="1" x="-2.54" y="88.9"/>
+<instance part="D3" gate="1" x="17.78" y="88.9"/>
 <instance part="D4" gate="1" x="111.76" y="73.66" rot="R90"/>
 <instance part="R2" gate="G$1" x="76.2" y="48.26" rot="R90"/>
 <instance part="R3" gate="G$1" x="76.2" y="35.56" rot="R90"/>
+<instance part="F1" gate="1" x="111.76" y="45.72" rot="R90"/>
+<instance part="F2" gate="1" x="12.7" y="81.28" rot="R270"/>
 </instances>
 <busses>
@@
 <net name="N$1" class="0">
 <segment>
-<wire x1="12.7" y1="88.9" x2="33.02" y2="88.9" width="0.1524" layer="91"/>
+<wire x1="25.4" y1="88.9" x2="33.02" y2="88.9" width="0.1524" layer="91"/>
 <pinref part="C1" gate="G$1" pin="1"/>
 <wire x1="33.02" y1="88.9" x2="111.76" y2="88.9" width="0.1524" layer="91"/>
-<wire x1="12.7" y1="86.36" x2="12.7" y2="88.9" width="0.1524" layer="91"/>
+<wire x1="25.4" y1="86.36" x2="25.4" y2="88.9" width="0.1524" layer="91"/>
 <wire x1="33.02" y1="88.9" x2="33.02" y2="63.5" width="0.1524" layer="91"/>
 <junction x="33.02" y="88.9"/>
@@
 <wire x1="111.76" y1="76.2" x2="111.76" y2="88.9" width="0.1524" layer="91"/>
 <pinref part="D3" gate="1" pin="C"/>
-<wire x1="0" y1="88.9" x2="12.7" y2="88.9" width="0.1524" layer="91"/>
-<junction x="12.7" y="88.9"/>
+<wire x1="20.32" y1="88.9" x2="25.4" y2="88.9" width="0.1524" layer="91"/>
+<junction x="25.4" y="88.9"/>
 </segment>
 </net>
@@
 <pinref part="SUPPLY1" gate="GND" pin="GND"/>
 <pinref part="C1" gate="G$1" pin="2"/>
-<wire x1="12.7" y1="76.2" x2="12.7" y2="78.74" width="0.1524" layer="91"/>
+<wire x1="25.4" y1="76.2" x2="25.4" y2="78.74" width="0.1524" layer="91"/>
 </segment>
 <segment>
 <pinref part="U$1" gate="G$2" pin="PAD"/>
 <pinref part="SUPPLY2" gate="GND" pin="GND"/>
-<wire x1="53.34" y1="40.64" x2="53.34" y2="35.56" width="0.1524" layer="91"/>
+<wire x1="53.34" y1="40.64" x2="53.34" y2="38.1" width="0.1524" layer="91"/>
 </segment>
 <segment>
@@
 <pinref part="R1" gate="G$1" pin="2"/>
 <wire x1="111.76" y1="58.42" x2="111.76" y2="53.34" width="0.1524" layer="91"/>
-<wire x1="111.76" y1="53.34" x2="111.76" y2="38.1" width="0.1524" layer="91"/>
+<wire x1="111.76" y1="53.34" x2="111.76" y2="50.8" width="0.1524" layer="91"/>
 <wire x1="93.98" y1="58.42" x2="111.76" y2="58.42" width="0.1524" layer="91"/>
 <junction x="111.76" y="58.42"/>
@@
 <junction x="111.76" y="53.34"/>
 <pinref part="R2" gate="G$1" pin="2"/>
+<pinref part="F1" gate="1" pin="2"/>
 </segment>
 </net>
@@
 </segment>
 </net>
+<net name="N$7" class="0">
+<segment>
+<pinref part="F2" gate="1" pin="1"/>
+<wire x1="12.7" y1="86.36" x2="12.7" y2="88.9" width="0.1524" layer="91"/>
+<pinref part="D3" gate="1" pin="A"/>
+<wire x1="12.7" y1="88.9" x2="15.24" y2="88.9" width="0.1524" layer="91"/>
+</segment>
+</net>
