File: board/board2/board2/board2.brd (EAGLE design)
At the start: 49.5 x 45.4 mm, 9 parts

Commit message: updated 2nd board
need to verify junctions are all in place
Parts:
- C1: value 0.1uF -> 4.7uF
- C2: value (none) -> 10uF
- C3: value (none) -> 0.1uF
- moved R2 34.2 mm to (8.89, 21.6), turned to 0 degrees
- moved C1 25.0 mm to (29.2, 12.7), turned to 270 degrees
- moved R3 21.0 mm to (6.35, 15.2)
- moved C2 20.8 mm to (20.3, 27.9)
- moved D1 13.1 mm to (29.2, 26.7), turned to 270 degrees
- moved U$2 11.5 mm to (8.89, 33.0), turned to 180 degrees
- moved U$1 8.98 mm to (16.5, 14.0), turned to 180 degrees
- moved C3 2.84 mm to (20.3, 20.3), turned to 270 degrees
Connections:
- removed net N$6: U$1.BST
- new net N$2: C3.+, U$1.BST
- net DGND: no longer C3.+
- net N$1: now also C1.-; no longer C2.-
- net N$3: now also C3.-, U$1.LX; no longer C1.-
- net N$4: now also C2.-; no longer C3.-
Routing:
- net N$5: track 92.0 -> 14.5 mm
- net DGND: track 73.4 -> 55.4 mm
- net N$2: track 0.00 -> 11.2 mm
- net N$1: track 5.81 -> 15.6 mm
- net N$3: track 38.0 -> 43.9 mm
- net N$4: track 43.8 -> 44.7 mm
Other:
- outline, holes or cut-outs redrawn
- board text added: "Dominik Kaukinen Colin Gagich hitchBOT 2014"

Commit message: 2nd board is complete
Parts:
- added LED2: (no value), led:SML0603
- added R1: 1k, rcl:R1206
Connections:
- new net N$6: LED2.A, R1.2
- net DGND: now also LED2.C
- net N$4: now also R1.1
Routing:
- net DGND: track 55.4 -> 77.5 mm, vias 0 -> 1
- net N$2: track 11.2 -> 18.8 mm, vias 0 -> 1
- net N$4: track 44.7 -> 51.5 mm
- net N$6: track 0.00 -> 4.18 mm
- net N$3: vias 0 -> 1
Other:
- board size 49.5 x 45.4 mm -> 38.1 x 46.7 mm
- board text added: "V 1.0"

Commit message: updated board2 for production
Parts:
- moved LED2 4.58 mm to (6.35, 5.08), turned to 180 degrees
- moved X1 3.81 mm to (16.5, -3.81)
- moved R1 2.54 mm to (5.08, 8.89)
- moved D1 1.27 mm to (29.2, 27.9)
Routing:
- net N$4: track 51.5 -> 60.6 mm, vias 0 -> 1
- net N$7: track 0.00 -> 6.35 mm
- net DGND: track 77.5 -> 73.9 mm
- net N$9: track 0.00 -> 2.54 mm
- net N$6: track 4.18 -> 2.44 mm
- net N$3: track 43.9 -> 45.2 mm
- net N$8: track 3.33 -> 2.08 mm
Other:
- board size 38.1 x 46.7 mm -> 35.5 x 45.4 mm
- board text added: "Dominik Kaukinen Colin Gagich USB Module hitchBOT 2014"
- board text added: "GND"
- board text added: "Vin"
- board text added: "Vout 5V"
- board text removed: "Dominik Kaukinen Colin Gagich hitchBOT 2014"
Changed lines of the file:
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@@
 <layer number="28" name="bValues" color="7" fill="1" visible="yes" active="yes"/>
 <layer number="29" name="tStop" color="7" fill="3" visible="no" active="yes"/>
-<layer number="30" name="bStop" color="7" fill="6" visible="no" active="yes"/>
+<layer number="30" name="bStop" color="7" fill="6" visible="yes" active="yes"/>
 <layer number="31" name="tCream" color="7" fill="4" visible="no" active="yes"/>
 <layer number="32" name="bCream" color="7" fill="5" visible="no" active="yes"/>
@@
 <board>
 <plain>
-<wire x1="-2.54" y1="-1.27" x2="35.54" y2="-1.27" width="0" layer="20"/>
-<wire x1="35.54" y1="-1.27" x2="35.54" y2="45.39" width="0" layer="20"/>
-<wire x1="35.54" y1="45.39" x2="-2.54" y2="45.39" width="0" layer="20"/>
-<wire x1="-2.54" y1="45.39" x2="-2.54" y2="-1.27" width="0" layer="20"/>
-<hole x="3.81" y="41.91" drill="5"/>
-<hole x="29.21" y="41.91" drill="5"/>
-<hole x="27.94" y="5.08" drill="5"/>
-<text x="12.7" y="38.1" size="1.016" layer="25">Dominik Kaukinen
+<wire x1="0" y1="0" x2="35.54" y2="0" width="0" layer="20"/>
+<wire x1="35.54" y1="0" x2="35.54" y2="45.39" width="0" layer="20"/>
+<wire x1="35.54" y1="45.39" x2="0" y2="45.39" width="0" layer="20"/>
+<wire x1="0" y1="45.39" x2="0" y2="0" width="0" layer="20"/>
+<hole x="3.81" y="41.91" drill="3.2"/>
+<hole x="30.48" y="41.91" drill="3.2"/>
+<hole x="30.48" y="5.08" drill="3.2"/>
+<text x="13.97" y="36.83" size="1.016" layer="25">Dominik Kaukinen
 Colin Gagich
+USB Module
 hitchBOT 2014
 </text>
-<text x="17.78" y="36.83" size="1.778" layer="25">V 1.0</text>
+<text x="16.51" y="35.56" size="1.778" layer="25">V 1.0</text>
+<rectangle x1="30.48" y1="7.62" x2="34.29" y2="11.43" layer="16"/>
+<rectangle x1="30.48" y1="13.97" x2="34.29" y2="17.78" layer="16"/>
+<text x="34.29" y="6.35" size="1.778" layer="22" rot="MR270">Vin</text>
+<text x="31.75" y="19.05" size="1.778" layer="22" rot="MR90">GND</text>
+<rectangle x1="30.48" y1="7.62" x2="34.29" y2="11.43" layer="30"/>
+<rectangle x1="30.48" y1="13.97" x2="34.29" y2="17.78" layer="30"/>
+<rectangle x1="1.27" y1="12.7" x2="6.35" y2="17.78" layer="16"/>
+<rectangle x1="1.27" y1="12.7" x2="6.35" y2="17.78" layer="30"/>
+<text x="5.08" y="30.48" size="1.778" layer="22" rot="MR270">Vout 5V</text>
 </plain>
 <attributes>
@@
 <element name="R2" library="rcl" package="M1206" value="9.53k" x="8.89" y="21.59"/>
 <element name="R3" library="rcl" package="M1206" value="49.9k" x="6.35" y="15.24"/>
-<element name="D1" library="diode" package="C4111-15" value="1N5908" x="29.21" y="26.67" rot="R270"/>
+<element name="D1" library="diode" package="C4111-15" value="1N5908" x="29.21" y="27.94" rot="R270"/>
 <element name="C3" library="c-trimm" package="3008" value="0.1uF" x="20.32" y="20.32" rot="R270">
 <attribute name="OC_NEWARK" value="unknown" x="-2.54" y="3.81" size="1.778" layer="27" rot="R270" display="off"/>
@@
 <element name="U$1" library="AO21282CI" package="AO21282CI" value="AO21282CI" x="16.51" y="13.97" rot="R180"/>
 <element name="U$2" library="AO21282CI" package="SRU1063" value="SRU1063" x="8.89" y="33.02" rot="R180"/>
-<element name="X1" library="con-amp" package="USB" value="" x="12.7" y="-3.81"/>
-<element name="LED2" library="led" package="SML0603" value="" x="2.54" y="2.54" rot="R90"/>
-<element name="R1" library="rcl" package="R1206" value="1k" x="2.54" y="8.89" rot="R270"/>
+<element name="X1" library="con-amp" package="USB" value="" x="16.51" y="-3.81"/>
+<element name="LED2" library="led" package="SML0603" value="" x="6.35" y="5.08" rot="R180"/>
+<element name="R1" library="rcl" package="R1206" value="1k" x="5.08" y="8.89" rot="R270"/>
 </elements>
 <signals>
@@
 <wire x1="20.32" y1="19.05" x2="20.32" y2="18.445" width="1.016" layer="1"/>
 <wire x1="29.21" y1="33.02" x2="13.39" y2="33.02" width="1.27" layer="1"/>
-<wire x1="29.21" y1="33.02" x2="29.21" y2="34.29" width="0.1524" layer="1"/>
+<wire x1="29.21" y1="33.02" x2="29.21" y2="35.56" width="0.1524" layer="1"/>
 <wire x1="17.46" y1="12.77" x2="19.05" y2="12.77" width="0.6096" layer="1"/>
 <wire x1="19.05" y1="12.77" x2="19.05" y2="13.97" width="0.6096" layer="1"/>
@@
 <wire x1="15.24" y1="21.59" x2="21.59" y2="27.94" width="1.016" layer="1"/>
 <wire x1="21.59" y1="27.94" x2="22.195" y2="27.94" width="1.016" layer="1"/>
-<wire x1="21.59" y1="13.97" x2="16.51" y2="8.89" width="1.016" layer="16"/>
+<wire x1="21.59" y1="13.97" x2="20.32" y2="8.89" width="1.016" layer="16"/>
 <wire x1="29.21" y1="13.97" x2="21.59" y2="13.97" width="1.016" layer="16"/>
-<wire x1="16.51" y1="8.89" x2="16.2001" y2="9.1801" width="0.1524" layer="16"/>
+<wire x1="20.32" y1="8.89" x2="20.0101" y2="9.1801" width="0.1524" layer="16"/>
 <wire x1="29.21" y1="13.97" x2="29.21" y2="14.575" width="0.1524" layer="16"/>
 <wire x1="29.21" y1="14.575" x2="29.21" y2="16.51" width="1.016" layer="1"/>
-<wire x1="29.21" y1="16.51" x2="29.21" y2="19.05" width="1.016" layer="1"/>
+<wire x1="29.21" y1="16.51" x2="29.21" y2="20.32" width="1.016" layer="1"/>
 <wire x1="29.21" y1="16.51" x2="16.51" y2="16.51" width="1.016" layer="1"/>
 <contactref element="LED2" pad="C"/>
-<wire x1="2.54" y1="1.79" x2="5.08" y2="1.79" width="0.8128" layer="1"/>
-<wire x1="5.08" y1="1.79" x2="5.08" y2="1.27" width="0.8128" layer="1"/>
-<via x="5.08" y="1.27" extent="1-16" drill="0.6" shape="square"/>
-<wire x1="5.08" y1="1.27" x2="16.2001" y2="1.27" width="0.8128" layer="16"/>
-<wire x1="16.2001" y1="1.27" x2="16.2001" y2="9.1801" width="0.8128" layer="16"/>
+<wire x1="7.1" y1="5.08" x2="11.43" y2="3.06" width="0.8128" layer="1"/>
+<wire x1="11.43" y1="3.06" x2="15.24" y2="5.08" width="0.8128" layer="1"/>
+<via x="15.24" y="5.08" extent="1-16" drill="0.6" shape="square"/>
+<wire x1="15.24" y1="5.08" x2="18.7401" y2="7.62" width="0.8128" layer="16"/>
+<wire x1="18.7401" y1="7.62" x2="20.0101" y2="9.1801" width="0.8128" layer="16"/>
+<wire x1="29.21" y1="13.97" x2="31.75" y2="13.97" width="1.016" layer="16"/>
+<wire x1="31.75" y1="13.97" x2="31.75" y2="15.24" width="1.016" layer="16"/>
 </signal>
 <signal name="N$4">
@@
 <wire x1="8.89" y1="33.02" x2="8.89" y2="27.94" width="1.016" layer="1"/>
 <wire x1="8.89" y1="27.94" x2="18.445" y2="27.94" width="1.016" layer="1"/>
-<wire x1="9.1999" y1="9.1801" x2="8.89" y2="9.1801" width="1.016" layer="1"/>
+<wire x1="13.0099" y1="9.1801" x2="8.89" y2="9.1801" width="1.016" layer="1"/>
 <wire x1="8.89" y1="9.1801" x2="8.89" y2="12.7" width="1.016" layer="1"/>
 <wire x1="8.89" y1="12.7" x2="5.08" y2="12.7" width="1.016" layer="1"/>
@@
 <wire x1="4.95" y1="12.7" x2="4.95" y2="15.24" width="1.016" layer="1"/>
 <contactref element="R1" pad="1"/>
-<wire x1="5.08" y1="12.7" x2="2.54" y2="10.16" width="0.8128" layer="1"/>
-<wire x1="2.54" y1="10.16" x2="2.54" y2="10.312" width="0.1524" layer="1"/>
+<wire x1="5.08" y1="12.7" x2="5.08" y2="10.16" width="0.8128" layer="1"/>
+<wire x1="5.08" y1="10.16" x2="5.08" y2="10.312" width="0.1524" layer="1"/>
+<via x="10.16" y="12.7" extent="1-16" drill="0.6" shape="square"/>
+<wire x1="8.89" y1="12.7" x2="10.16" y2="12.7" width="1.016" layer="1"/>
+<wire x1="10.16" y1="12.7" x2="6.35" y2="12.7" width="1.016" layer="16"/>
+<wire x1="6.35" y1="12.7" x2="6.35" y2="13.97" width="1.016" layer="16"/>
 </signal>
 <signal name="N$5">
@@
 <contactref element="X1" pad="3"/>
 <contactref element="X1" pad="2"/>
-<wire x1="13.97" y1="8.89" x2="11.43" y2="8.89" width="1.016" layer="1"/>
-<wire x1="11.43" y1="8.89" x2="11.7" y2="9.1801" width="0.254" layer="1"/>
-<wire x1="13.97" y1="8.89" x2="13.7" y2="9.1801" width="0.254" layer="1"/>
+<wire x1="16.51" y1="8.89" x2="15.51" y2="9.1801" width="0.254" layer="1"/>
+<wire x1="16.51" y1="8.89" x2="17.51" y2="9.1801" width="0.254" layer="1"/>
 </signal>
 <signal name="N$2">
@@
 <contactref element="LED2" pad="A"/>
 <contactref element="R1" pad="2"/>
-<wire x1="2.54" y1="3.29" x2="2.54" y2="7.468" width="0.8128" layer="1"/>
+<wire x1="5.6" y1="5.08" x2="5.08" y2="7.468" width="0.8128" layer="1"/>
+</signal>
+<signal name="N$7">
+<wire x1="29.21" y1="11.43" x2="31.75" y2="11.43" width="1.016" layer="16"/>
+<wire x1="31.75" y1="11.43" x2="31.75" y2="10.16" width="1.016" layer="16"/>
+<wire x1="29.21" y1="10.16" x2="31.75" y2="10.16" width="1.016" layer="16"/>
+</signal>
+<signal name="N$9">
+<wire x1="15.24" y1="8.89" x2="17.78" y2="8.89" width="1.016" layer="1"/>
 </signal>
 </signals>
