File: board/board2/board2/board2.sch (EAGLE design)
At the start: 9 parts

Commit message: 2nd board is complete
Parts:
- added LED2: (no value), led:LEDSML0603
- added R1: 1k, rcl:R-EU_R1206
Connections:
- new net N$6: LED2.A, R1.2
- net DGND: now also LED2.C
- net N$4: now also R1.1
Changed lines of the file:
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@@
 <part name="U$2" library="AO21282CI" deviceset="SRU1063" device=""/>
 <part name="X1" library="con-amp" deviceset="USB-787616" device=""/>
+<part name="LED2" library="led" deviceset="LED" device="SML0603"/>
+<part name="R1" library="rcl" deviceset="R-EU_" device="R1206" value="1k"/>
 </parts>
 <sheets>
@@
 <instance part="U$2" gate="G$1" x="53.34" y="10.16"/>
 <instance part="X1" gate="G$1" x="142.24" y="12.7"/>
+<instance part="LED2" gate="G$1" x="149.86" y="38.1" rot="R180"/>
+<instance part="R1" gate="G$1" x="152.4" y="30.48" rot="R90"/>
 </instances>
 <busses>
@@
 <wire x1="-30.48" y1="27.94" x2="-30.48" y2="25.4" width="0.1524" layer="91"/>
 <wire x1="-30.48" y1="25.4" x2="-60.96" y2="25.4" width="0.1524" layer="91"/>
+<pinref part="LED2" gate="G$1" pin="C"/>
+<wire x1="149.86" y1="43.18" x2="149.86" y2="63.5" width="0.1524" layer="91"/>
+<wire x1="149.86" y1="63.5" x2="124.46" y2="63.5" width="0.1524" layer="91"/>
 </segment>
 </net>
@@
 <wire x1="81.28" y1="10.16" x2="81.28" y2="30.48" width="0.1524" layer="91"/>
 <pinref part="C2" gate="G$1" pin="A"/>
-<wire x1="124.46" y1="40.64" x2="124.46" y2="17.78" width="0.1524" layer="91"/>
+<wire x1="124.46" y1="40.64" x2="124.46" y2="25.4" width="0.1524" layer="91"/>
+<wire x1="124.46" y1="25.4" x2="124.46" y2="17.78" width="0.1524" layer="91"/>
 <wire x1="124.46" y1="17.78" x2="124.46" y2="10.16" width="0.1524" layer="91"/>
 <wire x1="124.46" y1="10.16" x2="81.28" y2="10.16" width="0.1524" layer="91"/>
 <pinref part="X1" gate="G$1" pin="1"/>
 <wire x1="137.16" y1="17.78" x2="124.46" y2="17.78" width="0.1524" layer="91"/>
+<wire x1="152.4" y1="25.4" x2="124.46" y2="25.4" width="0.1524" layer="91"/>
+<pinref part="R1" gate="G$1" pin="1"/>
 </segment>
 </net>
@@
 </segment>
 </net>
+<net name="N$6" class="0">
+<segment>
+<pinref part="LED2" gate="G$1" pin="A"/>
+<pinref part="R1" gate="G$1" pin="2"/>
+<wire x1="152.4" y1="35.56" x2="149.86" y2="35.56" width="0.1524" layer="91"/>
+</segment>
+</net>
