File: board/Boards/Power Distribution/Power Distribution.brd (EAGLE design)
At the start: 45.7 x 72.1 mm, 14 parts

Commit message: new pads
Parts:
- added C1: (no value), resistor:E2,5-6
- added TP10, TP11, TP5, TP6, TP7, TP8, TP9: TP2P2-38-17, testpad:P2-38-17
- added TP12, TP13: TPTP20SQ, testpad:TP20SQ
- TP1, TP2, TP3, TP4: value TP5P5-25-17 -> TP2P2-38-17; device testpad:P5-25-17 -> testpad:P2-38-17
- moved TP3 91.6 mm to (2.54, -22.9), turned to 0 degrees
- moved TP1 61.7 mm to (2.54, -5.08), turned to 0 degrees
- moved TP4 56.8 mm to (2.54, -31.8), turned to 0 degrees
- moved TP2 55.8 mm to (2.54, -14.0), turned to 0 degrees
Connections:
- net GND: no longer TP3.TP-1, TP3.TP-2, TP3.TP-3, TP3.TP-4, TP3.TP-5, TP4.TP-1, TP4.TP-2, TP4.TP-3, TP4.TP-4, TP4.TP-5
- net N$6: no longer TP1.TP-1, TP1.TP-2, TP1.TP-3, TP1.TP-4, TP1.TP-5, TP2.TP-1, TP2.TP-2, TP2.TP-3, TP2.TP-4, TP2.TP-5
Changed lines of the file:
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@@
 <element name="U$9" library="Diodes" package="DO-214AB" value="DO-214AB" x="26.67" y="63.5"/>
 <element name="U$10" library="Diodes" package="DO-214AB" value="DO-214AB" x="26.67" y="7.62"/>
-<element name="TP1" library="testpad" package="P5-25-17" value="TP5P5-25-17" x="39.37" y="44.45" rot="R90">
-<attribute name="TP_SIGNAL_NAME" value="" x="92.71" y="68.58" size="1.778" layer="27" rot="R90" display="off"/>
+<element name="TP1" library="testpad" package="P2-38-17" value="TP2P2-38-17" x="2.54" y="-5.08">
+<attribute name="TP_SIGNAL_NAME" value="" x="2.54" y="-5.08" size="1.778" layer="27" display="off"/>
 </element>
-<element name="TP2" library="testpad" package="P5-25-17" value="TP5P5-25-17" x="39.37" y="27.94" rot="R90">
-<attribute name="TP_SIGNAL_NAME" value="" x="92.71" y="71.12" size="1.778" layer="27" rot="R90" display="off"/>
+<element name="TP2" library="testpad" package="P2-38-17" value="TP2P2-38-17" x="2.54" y="-13.97">
+<attribute name="TP_SIGNAL_NAME" value="" x="2.54" y="-13.97" size="1.778" layer="27" display="off"/>
 </element>
-<element name="TP3" library="testpad" package="P5-25-17" value="TP5P5-25-17" x="39.37" y="60.96" rot="R270">
-<attribute name="TP_SIGNAL_NAME" value="" x="-21.59" y="36.83" size="1.778" layer="27" rot="R270" display="off"/>
+<element name="TP3" library="testpad" package="P2-38-17" value="TP2P2-38-17" x="2.54" y="-22.86">
+<attribute name="TP_SIGNAL_NAME" value="" x="2.54" y="-22.86" size="1.778" layer="27" display="off"/>
 </element>
-<element name="TP4" library="testpad" package="P5-25-17" value="TP5P5-25-17" x="39.37" y="11.43" rot="R90">
-<attribute name="TP_SIGNAL_NAME" value="" x="100.33" y="54.61" size="1.778" layer="27" rot="R90" display="off"/>
+<element name="TP4" library="testpad" package="P2-38-17" value="TP2P2-38-17" x="2.54" y="-31.75">
+<attribute name="TP_SIGNAL_NAME" value="" x="2.54" y="-31.75" size="1.778" layer="27" display="off"/>
+</element>
+<element name="TP5" library="testpad" package="P2-38-17" value="TP2P2-38-17" x="2.54" y="-40.64">
+<attribute name="TP_SIGNAL_NAME" value="" x="2.54" y="-40.64" size="1.778" layer="27" display="off"/>
+</element>
+<element name="TP6" library="testpad" package="P2-38-17" value="TP2P2-38-17" x="2.54" y="-49.53">
+<attribute name="TP_SIGNAL_NAME" value="" x="2.54" y="-49.53" size="1.778" layer="27" display="off"/>
+</element>
+<element name="TP7" library="testpad" package="P2-38-17" value="TP2P2-38-17" x="2.54" y="-58.42">
+<attribute name="TP_SIGNAL_NAME" value="" x="2.54" y="-58.42" size="1.778" layer="27" display="off"/>
+</element>
+<element name="TP8" library="testpad" package="P2-38-17" value="TP2P2-38-17" x="2.54" y="-67.31">
+<attribute name="TP_SIGNAL_NAME" value="" x="2.54" y="-67.31" size="1.778" layer="27" display="off"/>
+</element>
+<element name="TP9" library="testpad" package="P2-38-17" value="TP2P2-38-17" x="2.54" y="-76.2">
+<attribute name="TP_SIGNAL_NAME" value="" x="2.54" y="-76.2" size="1.778" layer="27" display="off"/>
+</element>
+<element name="TP10" library="testpad" package="P2-38-17" value="TP2P2-38-17" x="2.54" y="-85.09">
+<attribute name="TP_SIGNAL_NAME" value="" x="2.54" y="-85.09" size="1.778" layer="27" display="off"/>
+</element>
+<element name="TP11" library="testpad" package="P2-38-17" value="TP2P2-38-17" x="2.54" y="-93.98">
+<attribute name="TP_SIGNAL_NAME" value="" x="2.54" y="-93.98" size="1.778" layer="27" display="off"/>
+</element>
+<element name="C1" library="resistor" package="E2,5-6" value="" x="2.54" y="-101.6"/>
+<element name="TP12" library="testpad" package="TP20SQ" value="TPTP20SQ" x="1.27" y="-107.95">
+<attribute name="TP_SIGNAL_NAME" value="" x="1.27" y="-107.95" size="1.778" layer="27" display="off"/>
+</element>
+<element name="TP13" library="testpad" package="TP20SQ" value="TPTP20SQ" x="1.27" y="-113.03">
+<attribute name="TP_SIGNAL_NAME" value="" x="1.27" y="-113.03" size="1.778" layer="27" display="off"/>
 </element>
 </elements>
@@
 <contactref element="U$5" pad="GNDL"/>
 <contactref element="U$5" pad="GNDR"/>
-<contactref element="TP3" pad="TP-1"/>
-<contactref element="TP3" pad="TP-2"/>
-<contactref element="TP3" pad="TP-3"/>
-<contactref element="TP3" pad="TP-4"/>
-<contactref element="TP3" pad="TP-5"/>
-<contactref element="TP4" pad="TP-1"/>
-<contactref element="TP4" pad="TP-2"/>
-<contactref element="TP4" pad="TP-3"/>
-<contactref element="TP4" pad="TP-4"/>
-<contactref element="TP4" pad="TP-5"/>
-<wire x1="39.37" y1="63.5" x2="39.37" y2="66.04" width="0" layer="19" extent="1-1"/>
-<wire x1="39.37" y1="60.96" x2="39.37" y2="63.5" width="0" layer="19" extent="1-1"/>
-<wire x1="39.37" y1="58.42" x2="39.37" y2="60.96" width="0" layer="19" extent="1-1"/>
-<wire x1="39.37" y1="55.88" x2="39.37" y2="58.42" width="0" layer="19" extent="1-1"/>
-<wire x1="13.14" y1="65.6" x2="39.37" y2="66.04" width="0" layer="19" extent="1-1"/>
 <wire x1="13.14" y1="61.4" x2="13.14" y2="65.6" width="0" layer="19" extent="1-1"/>
 <wire x1="13.14" y1="51.63" x2="13.14" y2="61.4" width="0" layer="19" extent="1-1"/>
@@
 <wire x1="13.14" y1="9.72" x2="13.14" y2="19.49" width="0" layer="19" extent="1-1"/>
 <wire x1="13.14" y1="5.52" x2="13.14" y2="9.72" width="0" layer="19" extent="1-1"/>
-<wire x1="39.37" y1="8.89" x2="13.14" y2="9.72" width="0" layer="19" extent="1-1"/>
-<wire x1="39.37" y1="11.43" x2="39.37" y2="8.89" width="0" layer="19" extent="1-1"/>
-<wire x1="39.37" y1="13.97" x2="39.37" y2="11.43" width="0" layer="19" extent="1-1"/>
-<wire x1="39.37" y1="16.51" x2="39.37" y2="13.97" width="0" layer="19" extent="1-1"/>
-<wire x1="39.37" y1="6.35" x2="39.37" y2="8.89" width="0" layer="19" extent="1-1"/>
 </signal>
 <signal name="N$1">
@@
 <contactref element="U$8" pad="OUT"/>
 <contactref element="U$7" pad="OUT"/>
-<contactref element="TP1" pad="TP-1"/>
-<contactref element="TP1" pad="TP-2"/>
-<contactref element="TP1" pad="TP-3"/>
-<contactref element="TP1" pad="TP-4"/>
-<contactref element="TP1" pad="TP-5"/>
-<contactref element="TP2" pad="TP-1"/>
-<contactref element="TP2" pad="TP-2"/>
-<contactref element="TP2" pad="TP-3"/>
-<contactref element="TP2" pad="TP-4"/>
-<contactref element="TP2" pad="TP-5"/>
 <wire x1="29.972" y1="49.53" x2="29.972" y2="63.5" width="0" layer="19" extent="1-1"/>
-<wire x1="39.37" y1="49.53" x2="29.972" y2="49.53" width="0" layer="19" extent="1-1"/>
-<wire x1="39.37" y1="46.99" x2="39.37" y2="49.53" width="0" layer="19" extent="1-1"/>
-<wire x1="39.37" y1="44.45" x2="39.37" y2="46.99" width="0" layer="19" extent="1-1"/>
-<wire x1="39.37" y1="41.91" x2="39.37" y2="44.45" width="0" layer="19" extent="1-1"/>
-<wire x1="39.37" y1="39.37" x2="39.37" y2="41.91" width="0" layer="19" extent="1-1"/>
-<wire x1="39.37" y1="33.02" x2="39.37" y2="39.37" width="0" layer="19" extent="1-1"/>
-<wire x1="39.37" y1="30.48" x2="39.37" y2="33.02" width="0" layer="19" extent="1-1"/>
-<wire x1="39.37" y1="27.94" x2="39.37" y2="30.48" width="0" layer="19" extent="1-1"/>
-<wire x1="39.37" y1="25.4" x2="39.37" y2="27.94" width="0" layer="19" extent="1-1"/>
-<wire x1="39.37" y1="22.86" x2="39.37" y2="25.4" width="0" layer="19" extent="1-1"/>
-<wire x1="29.972" y1="21.59" x2="39.37" y2="22.86" width="0" layer="19" extent="1-1"/>
-<wire x1="29.972" y1="35.56" x2="39.37" y2="33.02" width="0" layer="19" extent="1-1"/>
+<wire x1="29.972" y1="35.56" x2="29.972" y2="49.53" width="0" layer="19" extent="1-1"/>
+<wire x1="29.972" y1="21.59" x2="29.972" y2="35.56" width="0" layer="19" extent="1-1"/>
 <wire x1="29.972" y1="7.62" x2="29.972" y2="21.59" width="0" layer="19" extent="1-1"/>
 </signal>
