File: board/Boards/Power Distribution/Power Distribution.brd (EAGLE design)
At the start: 48.2 x 84.8 mm, 24 parts

Commit message: poly's added
Parts:
- turned C1 to 270 degrees
Routing:
- net GND: track 0.00 -> 2.54 mm, vias 0 -> 1
- added copper zone on layer 16, net GND
- added copper zone on layer 1, net N$1
- added copper zone on layer 1, net N$2
- added copper zone on layer 1, net N$3
- added copper zone on layer 1, net N$4
- added copper zone on layer 1, net N$5
- added copper zone on layer 1, net N$6
Changed lines of the file:
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@@
 <attribute name="TP_SIGNAL_NAME" value="" x="100.33" y="-17.78" size="1.778" layer="27" display="off"/>
 </element>
-<element name="C1" library="resistor" package="E2,5-6" value="" x="27.94" y="78.74" rot="R180"/>
+<element name="C1" library="resistor" package="E2,5-6" value="" x="27.94" y="78.74" rot="R270"/>
 <element name="TP12" library="testpad" package="TP20SQ" value="TPTP20SQ" x="19.05" y="78.74">
 <attribute name="TP_SIGNAL_NAME" value="" x="57.15" y="8.89" size="1.778" layer="27" display="off"/>
@@
 <contactref element="TP9" pad="TP-2"/>
 <contactref element="TP10" pad="TP-2"/>
-<wire x1="42.545" y1="72.39" x2="42.545" y2="78.74" width="0" layer="19" extent="1-1"/>
-<wire x1="42.545" y1="64.77" x2="42.545" y2="72.39" width="0" layer="19" extent="1-1"/>
-<wire x1="42.545" y1="58.42" x2="42.545" y2="64.77" width="0" layer="19" extent="1-1"/>
-<wire x1="42.545" y1="50.8" x2="42.545" y2="58.42" width="0" layer="19" extent="1-1"/>
-<wire x1="42.545" y1="44.45" x2="42.545" y2="50.8" width="0" layer="19" extent="1-1"/>
-<wire x1="42.545" y1="36.83" x2="42.545" y2="44.45" width="0" layer="19" extent="1-1"/>
-<wire x1="42.545" y1="30.48" x2="42.545" y2="36.83" width="0" layer="19" extent="1-1"/>
-<wire x1="42.545" y1="22.86" x2="42.545" y2="30.48" width="0" layer="19" extent="1-1"/>
-<wire x1="42.545" y1="16.51" x2="42.545" y2="22.86" width="0" layer="19" extent="1-1"/>
-<wire x1="40.64" y1="9.525" x2="42.545" y2="16.51" width="0" layer="19" extent="1-1"/>
-<wire x1="26.67" y1="78.74" x2="42.545" y2="78.74" width="0" layer="19" extent="1-1"/>
-<wire x1="12.7" y1="78.74" x2="26.67" y2="78.74" width="0" layer="19" extent="1-1"/>
-<wire x1="13.14" y1="70.68" x2="12.7" y2="78.74" width="0" layer="19" extent="1-1"/>
-<wire x1="13.14" y1="66.48" x2="13.14" y2="70.68" width="0" layer="19" extent="1-1"/>
-<wire x1="13.14" y1="55.44" x2="13.14" y2="66.48" width="0" layer="19" extent="1-1"/>
-<wire x1="13.14" y1="51.24" x2="13.14" y2="55.44" width="0" layer="19" extent="1-1"/>
-<wire x1="13.14" y1="40.2" x2="13.14" y2="51.24" width="0" layer="19" extent="1-1"/>
-<wire x1="13.14" y1="36" x2="13.14" y2="40.2" width="0" layer="19" extent="1-1"/>
-<wire x1="13.14" y1="24.96" x2="13.14" y2="36" width="0" layer="19" extent="1-1"/>
-<wire x1="13.14" y1="20.76" x2="13.14" y2="24.96" width="0" layer="19" extent="1-1"/>
-<wire x1="13.14" y1="9.72" x2="13.14" y2="20.76" width="0" layer="19" extent="1-1"/>
-<wire x1="13.14" y1="5.52" x2="13.14" y2="9.72" width="0" layer="19" extent="1-1"/>
+<polygon width="0.4064" layer="16" isolate="0.4064">
+<vertex x="-1.27" y="86.36"/>
+<vertex x="49.53" y="86.36"/>
+<vertex x="49.53" y="-1.27"/>
+<vertex x="-1.27" y="-1.27"/>
+</polygon>
+<wire x1="12.7" y1="78.74" x2="10.16" y2="78.74" width="0.4064" layer="1"/>
+<via x="10.16" y="78.74" extent="1-16" drill="0.6"/>
 </signal>
 <signal name="N$1">
@@
 <contactref element="U$5" pad="POWERR"/>
 <contactref element="U$6" pad="IN"/>
-<wire x1="17.34" y1="9.72" x2="24.638" y2="7.62" width="0" layer="19" extent="1-1"/>
-<wire x1="17.34" y1="5.52" x2="17.34" y2="9.72" width="0" layer="19" extent="1-1"/>
+<polygon width="0.4064" layer="1" isolate="0.4064">
+<vertex x="1.27" y="13.97"/>
+<vertex x="26.67" y="13.97"/>
+<vertex x="26.67" y="1.27"/>
+<vertex x="1.27" y="1.27"/>
+</polygon>
 </signal>
 <signal name="N$2">
@@
 <contactref element="U$1" pad="POWERR"/>
 <contactref element="U$7" pad="IN"/>
-<wire x1="17.34" y1="24.96" x2="24.638" y2="22.86" width="0" layer="19" extent="1-1"/>
-<wire x1="17.34" y1="20.76" x2="17.34" y2="24.96" width="0" layer="19" extent="1-1"/>
+<polygon width="0.4064" layer="1" isolate="0.4064">
+<vertex x="1.27" y="29.21"/>
+<vertex x="26.67" y="29.21"/>
+<vertex x="26.67" y="16.51"/>
+<vertex x="1.27" y="16.51"/>
+</polygon>
 </signal>
 <signal name="N$3">
@@
 <contactref element="U$2" pad="POWERR"/>
 <contactref element="U$8" pad="IN"/>
-<wire x1="17.34" y1="40.2" x2="24.638" y2="38.1" width="0" layer="19" extent="1-1"/>
-<wire x1="17.34" y1="36" x2="17.34" y2="40.2" width="0" layer="19" extent="1-1"/>
+<polygon width="0.4064" layer="1" isolate="0.4064">
+<vertex x="1.27" y="44.45"/>
+<vertex x="26.67" y="44.45"/>
+<vertex x="26.67" y="31.75"/>
+<vertex x="1.27" y="31.75"/>
+</polygon>
 </signal>
 <signal name="N$4">
@@
 <contactref element="U$3" pad="POWERR"/>
 <contactref element="U$9" pad="IN"/>
-<wire x1="17.34" y1="51.24" x2="17.34" y2="55.44" width="0" layer="19" extent="1-1"/>
-<wire x1="17.34" y1="55.44" x2="24.638" y2="53.34" width="0" layer="19" extent="1-1"/>
+<polygon width="0.4064" layer="1" isolate="0.4064">
+<vertex x="1.27" y="59.69"/>
+<vertex x="26.67" y="59.69"/>
+<vertex x="26.67" y="46.99"/>
+<vertex x="1.27" y="46.99"/>
+</polygon>
 </signal>
 <signal name="N$5">
@@
 <contactref element="U$4" pad="POWERR"/>
 <contactref element="U$10" pad="IN"/>
-<wire x1="17.34" y1="70.68" x2="24.638" y2="68.58" width="0" layer="19" extent="1-1"/>
-<wire x1="17.34" y1="66.48" x2="17.34" y2="70.68" width="0" layer="19" extent="1-1"/>
+<polygon width="0.4064" layer="1" isolate="0.4064">
+<vertex x="26.67" y="74.93"/>
+<vertex x="26.67" y="62.23"/>
+<vertex x="-1.27" y="62.23"/>
+<vertex x="-1.27" y="74.93"/>
+</polygon>
 </signal>
 <signal name="N$6">
@@
 <contactref element="TP9" pad="TP-1"/>
 <contactref element="TP10" pad="TP-1"/>
-<wire x1="38.735" y1="72.39" x2="38.735" y2="78.74" width="0" layer="19" extent="1-1"/>
-<wire x1="38.735" y1="64.77" x2="38.735" y2="72.39" width="0" layer="19" extent="1-1"/>
-<wire x1="38.735" y1="58.42" x2="38.735" y2="64.77" width="0" layer="19" extent="1-1"/>
-<wire x1="38.735" y1="50.8" x2="38.735" y2="58.42" width="0" layer="19" extent="1-1"/>
-<wire x1="38.735" y1="44.45" x2="38.735" y2="50.8" width="0" layer="19" extent="1-1"/>
-<wire x1="38.735" y1="36.83" x2="38.735" y2="44.45" width="0" layer="19" extent="1-1"/>
-<wire x1="38.735" y1="30.48" x2="38.735" y2="36.83" width="0" layer="19" extent="1-1"/>
-<wire x1="31.242" y1="38.1" x2="38.735" y2="36.83" width="0" layer="19" extent="1-1"/>
-<wire x1="38.735" y1="22.86" x2="38.735" y2="30.48" width="0" layer="19" extent="1-1"/>
-<wire x1="38.735" y1="16.51" x2="38.735" y2="22.86" width="0" layer="19" extent="1-1"/>
-<wire x1="31.242" y1="22.86" x2="38.735" y2="22.86" width="0" layer="19" extent="1-1"/>
-<wire x1="31.242" y1="53.34" x2="38.735" y2="50.8" width="0" layer="19" extent="1-1"/>
-<wire x1="29.21" y1="78.74" x2="38.735" y2="78.74" width="0" layer="19" extent="1-1"/>
-<wire x1="31.242" y1="68.58" x2="38.735" y2="72.39" width="0" layer="19" extent="1-1"/>
-<wire x1="40.64" y1="5.715" x2="38.735" y2="16.51" width="0" layer="19" extent="1-1"/>
-<wire x1="31.242" y1="7.62" x2="40.64" y2="5.715" width="0" layer="19" extent="1-1"/>
-<wire x1="19.05" y1="78.74" x2="29.21" y2="78.74" width="0" layer="19" extent="1-1"/>
+<polygon width="0.4064" layer="1" isolate="0.4064" rank="2">
+<vertex x="-1.27" y="86.36"/>
+<vertex x="49.53" y="86.36"/>
+<vertex x="49.53" y="-1.27"/>
+<vertex x="-1.27" y="-1.27"/>
+</polygon>
 </signal>
 </signals>
