File: board/Boards/Power Distribution/Power Distribution.sch (EAGLE design)
At the start: 14 parts

Commit message: new pads
Parts:
- added C1: (no value), resistor:CPOL-USE2.5-6
- added TP10, TP11, TP5, TP6, TP7, TP8, TP9: TP2P2-38-17, testpad:TP2P2-38-17
- added TP12, TP13: TPTP20SQ, testpad:TPTP20SQ
- TP1, TP2, TP3, TP4: value TP5P5-25-17 -> TP2P2-38-17; device testpad:TP5P5-25-17 -> testpad:TP2P2-38-17
Connections:
- net GND: now also C1.-; no longer TP3A.TP, TP3B.TP, TP3C.TP, TP3D.TP, TP3E.TP, TP4A.TP, TP4B.TP, TP4C.TP, TP4D.TP, TP4E.TP
- net N$6: now also C1.+; no longer TP1A.TP, TP1B.TP, TP1C.TP, TP1D.TP, TP1E.TP, TP2A.TP, TP2B.TP, TP2C.TP, TP2D.TP, TP2E.TP
Other:
- moved on the sheet: TP1A, TP1B, TP2A, TP2B, TP3A, TP3B, TP4A, TP4B
Changed lines of the file:
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@@
 <part name="U$9" library="Diodes" deviceset="DO-214AB" device=""/>
 <part name="U$10" library="Diodes" deviceset="DO-214AB" device=""/>
-<part name="TP1" library="testpad" deviceset="TP5" device="P5-25-17"/>
-<part name="TP2" library="testpad" deviceset="TP5" device="P5-25-17"/>
-<part name="TP3" library="testpad" deviceset="TP5" device="P5-25-17"/>
-<part name="TP4" library="testpad" deviceset="TP5" device="P5-25-17"/>
+<part name="TP1" library="testpad" deviceset="TP2" device="P2-38-17"/>
+<part name="TP2" library="testpad" deviceset="TP2" device="P2-38-17"/>
+<part name="TP3" library="testpad" deviceset="TP2" device="P2-38-17"/>
+<part name="TP4" library="testpad" deviceset="TP2" device="P2-38-17"/>
+<part name="TP5" library="testpad" deviceset="TP2" device="P2-38-17"/>
+<part name="TP6" library="testpad" deviceset="TP2" device="P2-38-17"/>
+<part name="TP7" library="testpad" deviceset="TP2" device="P2-38-17"/>
+<part name="TP8" library="testpad" deviceset="TP2" device="P2-38-17"/>
+<part name="TP9" library="testpad" deviceset="TP2" device="P2-38-17"/>
+<part name="TP10" library="testpad" deviceset="TP2" device="P2-38-17"/>
+<part name="TP11" library="testpad" deviceset="TP2" device="P2-38-17"/>
+<part name="C1" library="resistor" deviceset="CPOL-US" device="E2.5-6"/>
+<part name="TP12" library="testpad" deviceset="TP" device="TP20SQ"/>
+<part name="TP13" library="testpad" deviceset="TP" device="TP20SQ"/>
+<part name="SUPPLY2" library="supply2" deviceset="GND" device=""/>
+<part name="SUPPLY3" library="supply2" deviceset="GND" device=""/>
 </parts>
 <sheets>
@@
 <instance part="U$9" gate="G$1" x="35.56" y="38.1" rot="R270"/>
 <instance part="U$10" gate="G$1" x="35.56" y="15.24" rot="R270"/>
-<instance part="TP1" gate="A" x="71.12" y="104.14"/>
-<instance part="TP1" gate="B" x="76.2" y="104.14"/>
-<instance part="TP1" gate="C" x="81.28" y="104.14"/>
-<instance part="TP1" gate="D" x="86.36" y="104.14"/>
-<instance part="TP1" gate="E" x="91.44" y="104.14"/>
-<instance part="TP2" gate="A" x="71.12" y="91.44"/>
-<instance part="TP2" gate="B" x="76.2" y="91.44"/>
-<instance part="TP2" gate="C" x="81.28" y="91.44"/>
-<instance part="TP2" gate="D" x="86.36" y="91.44"/>
-<instance part="TP2" gate="E" x="91.44" y="91.44"/>
-<instance part="TP3" gate="A" x="35.56" y="0"/>
-<instance part="TP3" gate="B" x="40.64" y="0"/>
-<instance part="TP3" gate="C" x="45.72" y="0"/>
-<instance part="TP3" gate="D" x="50.8" y="0"/>
-<instance part="TP3" gate="E" x="55.88" y="0"/>
-<instance part="TP4" gate="A" x="35.56" y="-10.16"/>
-<instance part="TP4" gate="B" x="40.64" y="-10.16"/>
-<instance part="TP4" gate="C" x="45.72" y="-10.16"/>
-<instance part="TP4" gate="D" x="50.8" y="-10.16"/>
-<instance part="TP4" gate="E" x="55.88" y="-10.16"/>
+<instance part="TP1" gate="A" x="76.2" y="106.68"/>
+<instance part="TP1" gate="B" x="83.82" y="106.68"/>
+<instance part="TP2" gate="A" x="76.2" y="91.44"/>
+<instance part="TP2" gate="B" x="83.82" y="91.44"/>
+<instance part="TP3" gate="A" x="76.2" y="83.82"/>
+<instance part="TP3" gate="B" x="83.82" y="83.82"/>
+<instance part="TP4" gate="A" x="76.2" y="101.6"/>
+<instance part="TP4" gate="B" x="83.82" y="101.6"/>
+<instance part="TP5" gate="A" x="76.2" y="73.66"/>
+<instance part="TP5" gate="B" x="83.82" y="73.66"/>
+<instance part="TP6" gate="A" x="76.2" y="66.04"/>
+<instance part="TP6" gate="B" x="83.82" y="66.04"/>
+<instance part="TP7" gate="A" x="76.2" y="50.8"/>
+<instance part="TP7" gate="B" x="83.82" y="50.8"/>
+<instance part="TP8" gate="A" x="76.2" y="43.18"/>
+<instance part="TP8" gate="B" x="83.82" y="43.18"/>
+<instance part="TP9" gate="A" x="76.2" y="30.48"/>
+<instance part="TP9" gate="B" x="83.82" y="30.48"/>
+<instance part="TP10" gate="A" x="76.2" y="22.86"/>
+<instance part="TP10" gate="B" x="83.82" y="22.86"/>
+<instance part="TP11" gate="A" x="50.8" y="116.84"/>
+<instance part="TP11" gate="B" x="58.42" y="116.84"/>
+<instance part="C1" gate="G$1" x="63.5" y="109.22" rot="R180"/>
+<instance part="TP12" gate="G$1" x="10.16" y="119.38"/>
+<instance part="TP13" gate="G$1" x="17.78" y="119.38"/>
+<instance part="SUPPLY2" gate="GND" x="71.12" y="116.84"/>
+<instance part="SUPPLY3" gate="GND" x="99.06" y="7.62"/>
 </instances>
 <busses>
@@
 <junction x="25.4" y="33.02"/>
 <junction x="25.4" y="10.16"/>
-<wire x1="25.4" y1="5.08" x2="30.48" y2="5.08" width="0.1524" layer="91"/>
-<wire x1="30.48" y1="5.08" x2="30.48" y2="-2.54" width="0.1524" layer="91"/>
-<pinref part="TP3" gate="A" pin="TP"/>
-<wire x1="30.48" y1="-2.54" x2="35.56" y2="-2.54" width="0.1524" layer="91"/>
-<pinref part="TP3" gate="B" pin="TP"/>
-<wire x1="35.56" y1="-2.54" x2="40.64" y2="-2.54" width="0.1524" layer="91"/>
-<pinref part="TP3" gate="C" pin="TP"/>
-<wire x1="40.64" y1="-2.54" x2="45.72" y2="-2.54" width="0.1524" layer="91"/>
-<pinref part="TP3" gate="D" pin="TP"/>
-<wire x1="45.72" y1="-2.54" x2="50.8" y2="-2.54" width="0.1524" layer="91"/>
-<pinref part="TP3" gate="E" pin="TP"/>
-<wire x1="50.8" y1="-2.54" x2="55.88" y2="-2.54" width="0.1524" layer="91"/>
-<wire x1="30.48" y1="-2.54" x2="30.48" y2="-12.7" width="0.1524" layer="91"/>
-<pinref part="TP4" gate="A" pin="TP"/>
-<wire x1="30.48" y1="-12.7" x2="35.56" y2="-12.7" width="0.1524" layer="91"/>
-<pinref part="TP4" gate="B" pin="TP"/>
-<wire x1="35.56" y1="-12.7" x2="40.64" y2="-12.7" width="0.1524" layer="91"/>
-<pinref part="TP4" gate="C" pin="TP"/>
-<wire x1="40.64" y1="-12.7" x2="45.72" y2="-12.7" width="0.1524" layer="91"/>
-<pinref part="TP4" gate="D" pin="TP"/>
-<wire x1="45.72" y1="-12.7" x2="50.8" y2="-12.7" width="0.1524" layer="91"/>
-<pinref part="TP4" gate="E" pin="TP"/>
-<wire x1="50.8" y1="-12.7" x2="55.88" y2="-12.7" width="0.1524" layer="91"/>
+</segment>
+<segment>
+<pinref part="SUPPLY2" gate="GND" pin="GND"/>
+<pinref part="C1" gate="G$1" pin="-"/>
+<wire x1="71.12" y1="119.38" x2="63.5" y2="119.38" width="0.1524" layer="91"/>
+<wire x1="63.5" y1="119.38" x2="63.5" y2="114.3" width="0.1524" layer="91"/>
 </segment>
 </net>
@@
 <pinref part="U$10" gate="G$1" pin="OUT"/>
 <wire x1="55.88" y1="86.36" x2="55.88" y2="81.28" width="0.1524" layer="91"/>
-<wire x1="55.88" y1="81.28" x2="55.88" y2="60.96" width="0.1524" layer="91"/>
-<wire x1="55.88" y1="60.96" x2="55.88" y2="38.1" width="0.1524" layer="91"/>
-<wire x1="55.88" y1="38.1" x2="55.88" y2="15.24" width="0.1524" layer="91"/>
+<wire x1="55.88" y1="81.28" x2="55.88" y2="71.12" width="0.1524" layer="91"/>
+<wire x1="55.88" y1="71.12" x2="55.88" y2="60.96" width="0.1524" layer="91"/>
+<wire x1="55.88" y1="60.96" x2="55.88" y2="48.26" width="0.1524" layer="91"/>
+<wire x1="55.88" y1="48.26" x2="55.88" y2="38.1" width="0.1524" layer="91"/>
+<wire x1="55.88" y1="38.1" x2="55.88" y2="25.4" width="0.1524" layer="91"/>
+<wire x1="55.88" y1="25.4" x2="55.88" y2="15.24" width="0.1524" layer="91"/>
 <wire x1="55.88" y1="15.24" x2="45.72" y2="15.24" width="0.1524" layer="91"/>
 <pinref part="U$9" gate="G$1" pin="OUT"/>
@@
 <pinref part="U$7" gate="G$1" pin="OUT"/>
 <wire x1="45.72" y1="81.28" x2="55.88" y2="81.28" width="0.1524" layer="91"/>
-<pinref part="TP1" gate="A" pin="TP"/>
-<wire x1="55.88" y1="101.6" x2="71.12" y2="101.6" width="0.1524" layer="91"/>
-<pinref part="TP1" gate="B" pin="TP"/>
-<wire x1="71.12" y1="101.6" x2="76.2" y2="101.6" width="0.1524" layer="91"/>
-<pinref part="TP1" gate="C" pin="TP"/>
-<wire x1="76.2" y1="101.6" x2="81.28" y2="101.6" width="0.1524" layer="91"/>
-<pinref part="TP1" gate="D" pin="TP"/>
-<wire x1="81.28" y1="101.6" x2="86.36" y2="101.6" width="0.1524" layer="91"/>
-<pinref part="TP1" gate="E" pin="TP"/>
-<wire x1="86.36" y1="101.6" x2="91.44" y2="101.6" width="0.1524" layer="91"/>
-<pinref part="TP2" gate="A" pin="TP"/>
+<wire x1="55.88" y1="101.6" x2="63.5" y2="101.6" width="0.1524" layer="91"/>
+<wire x1="63.5" y1="101.6" x2="71.12" y2="101.6" width="0.1524" layer="91"/>
 <wire x1="55.88" y1="86.36" x2="71.12" y2="86.36" width="0.1524" layer="91"/>
-<wire x1="71.12" y1="86.36" x2="71.12" y2="88.9" width="0.1524" layer="91"/>
-<pinref part="TP2" gate="B" pin="TP"/>
-<wire x1="71.12" y1="88.9" x2="76.2" y2="88.9" width="0.1524" layer="91"/>
-<pinref part="TP2" gate="C" pin="TP"/>
-<wire x1="76.2" y1="88.9" x2="81.28" y2="88.9" width="0.1524" layer="91"/>
-<pinref part="TP2" gate="D" pin="TP"/>
-<wire x1="81.28" y1="88.9" x2="86.36" y2="88.9" width="0.1524" layer="91"/>
-<pinref part="TP2" gate="E" pin="TP"/>
-<wire x1="86.36" y1="88.9" x2="91.44" y2="88.9" width="0.1524" layer="91"/>
+<wire x1="55.88" y1="71.12" x2="71.12" y2="71.12" width="0.1524" layer="91"/>
+<wire x1="55.88" y1="48.26" x2="71.12" y2="48.26" width="0.1524" layer="91"/>
+<wire x1="55.88" y1="25.4" x2="71.12" y2="25.4" width="0.1524" layer="91"/>
+<pinref part="C1" gate="G$1" pin="+"/>
+<wire x1="63.5" y1="106.68" x2="63.5" y2="101.6" width="0.1524" layer="91"/>
 </segment>
 </net>

Commit message: everything wired up nice
Connections:
- net GND: now also TP10B.TP, TP11B.TP, TP13.TP, TP1B.TP, TP2B.TP, TP3B.TP, TP4B.TP, TP5B.TP, TP6B.TP, TP7B.TP, TP8B.TP, TP9B.TP
- net N$6: now also TP10A.TP, TP11A.TP, TP12.TP, TP1A.TP, TP2A.TP, TP3A.TP, TP4A.TP, TP5A.TP, TP6A.TP, TP7A.TP, TP8A.TP, TP9A.TP
Other:
- moved on the sheet: TP12, TP13
Changed lines of the file:
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@@
 <instance part="TP11" gate="B" x="58.42" y="116.84"/>
 <instance part="C1" gate="G$1" x="63.5" y="109.22" rot="R180"/>
-<instance part="TP12" gate="G$1" x="10.16" y="119.38"/>
-<instance part="TP13" gate="G$1" x="17.78" y="119.38"/>
+<instance part="TP12" gate="G$1" x="43.18" y="116.84"/>
+<instance part="TP13" gate="G$1" x="68.58" y="124.46"/>
 <instance part="SUPPLY2" gate="GND" x="71.12" y="116.84"/>
 <instance part="SUPPLY3" gate="GND" x="99.06" y="7.62"/>
@@
 <pinref part="SUPPLY2" gate="GND" pin="GND"/>
 <pinref part="C1" gate="G$1" pin="-"/>
-<wire x1="71.12" y1="119.38" x2="63.5" y2="119.38" width="0.1524" layer="91"/>
-<wire x1="63.5" y1="119.38" x2="63.5" y2="114.3" width="0.1524" layer="91"/>
+<wire x1="71.12" y1="119.38" x2="68.58" y2="119.38" width="0.1524" layer="91"/>
+<wire x1="68.58" y1="119.38" x2="63.5" y2="119.38" width="0.1524" layer="91"/>
+<wire x1="63.5" y1="119.38" x2="63.5" y2="116.84" width="0.1524" layer="91"/>
+<pinref part="TP11" gate="B" pin="TP"/>
+<wire x1="63.5" y1="116.84" x2="63.5" y2="114.3" width="0.1524" layer="91"/>
+<wire x1="58.42" y1="114.3" x2="60.96" y2="114.3" width="0.1524" layer="91"/>
+<wire x1="60.96" y1="114.3" x2="60.96" y2="116.84" width="0.1524" layer="91"/>
+<wire x1="60.96" y1="116.84" x2="63.5" y2="116.84" width="0.1524" layer="91"/>
+<pinref part="TP13" gate="G$1" pin="TP"/>
+<wire x1="68.58" y1="121.92" x2="68.58" y2="119.38" width="0.1524" layer="91"/>
+<junction x="63.5" y="116.84"/>
+<junction x="68.58" y="119.38"/>
+</segment>
+<segment>
+<pinref part="SUPPLY3" gate="GND" pin="GND"/>
+<wire x1="99.06" y1="10.16" x2="93.98" y2="10.16" width="0.1524" layer="91"/>
+<wire x1="93.98" y1="10.16" x2="93.98" y2="20.32" width="0.1524" layer="91"/>
+<pinref part="TP1" gate="B" pin="TP"/>
+<wire x1="93.98" y1="20.32" x2="93.98" y2="27.94" width="0.1524" layer="91"/>
+<wire x1="93.98" y1="27.94" x2="93.98" y2="40.64" width="0.1524" layer="91"/>
+<wire x1="93.98" y1="40.64" x2="93.98" y2="48.26" width="0.1524" layer="91"/>
+<wire x1="93.98" y1="48.26" x2="93.98" y2="63.5" width="0.1524" layer="91"/>
+<wire x1="93.98" y1="63.5" x2="93.98" y2="71.12" width="0.1524" layer="91"/>
+<wire x1="93.98" y1="71.12" x2="93.98" y2="81.28" width="0.1524" layer="91"/>
+<wire x1="93.98" y1="81.28" x2="93.98" y2="88.9" width="0.1524" layer="91"/>
+<wire x1="93.98" y1="88.9" x2="93.98" y2="99.06" width="0.1524" layer="91"/>
+<wire x1="93.98" y1="99.06" x2="93.98" y2="104.14" width="0.1524" layer="91"/>
+<wire x1="83.82" y1="104.14" x2="93.98" y2="104.14" width="0.1524" layer="91"/>
+<pinref part="TP4" gate="B" pin="TP"/>
+<wire x1="83.82" y1="99.06" x2="93.98" y2="99.06" width="0.1524" layer="91"/>
+<pinref part="TP2" gate="B" pin="TP"/>
+<wire x1="83.82" y1="88.9" x2="93.98" y2="88.9" width="0.1524" layer="91"/>
+<pinref part="TP3" gate="B" pin="TP"/>
+<wire x1="83.82" y1="81.28" x2="93.98" y2="81.28" width="0.1524" layer="91"/>
+<pinref part="TP5" gate="B" pin="TP"/>
+<wire x1="83.82" y1="71.12" x2="93.98" y2="71.12" width="0.1524" layer="91"/>
+<pinref part="TP6" gate="B" pin="TP"/>
+<wire x1="83.82" y1="63.5" x2="93.98" y2="63.5" width="0.1524" layer="91"/>
+<pinref part="TP7" gate="B" pin="TP"/>
+<wire x1="83.82" y1="48.26" x2="93.98" y2="48.26" width="0.1524" layer="91"/>
+<pinref part="TP8" gate="B" pin="TP"/>
+<wire x1="83.82" y1="40.64" x2="93.98" y2="40.64" width="0.1524" layer="91"/>
+<pinref part="TP9" gate="B" pin="TP"/>
+<wire x1="83.82" y1="27.94" x2="93.98" y2="27.94" width="0.1524" layer="91"/>
+<pinref part="TP10" gate="B" pin="TP"/>
+<wire x1="83.82" y1="20.32" x2="93.98" y2="20.32" width="0.1524" layer="91"/>
+<junction x="93.98" y="71.12"/>
+<junction x="93.98" y="81.28"/>
+<junction x="93.98" y="88.9"/>
+<junction x="93.98" y="99.06"/>
+<junction x="93.98" y="63.5"/>
+<junction x="93.98" y="48.26"/>
+<junction x="93.98" y="40.64"/>
+<junction x="93.98" y="20.32"/>
+<junction x="93.98" y="27.94"/>
 </segment>
 </net>
@@
 <wire x1="45.72" y1="81.28" x2="55.88" y2="81.28" width="0.1524" layer="91"/>
 <wire x1="55.88" y1="101.6" x2="63.5" y2="101.6" width="0.1524" layer="91"/>
-<wire x1="63.5" y1="101.6" x2="71.12" y2="101.6" width="0.1524" layer="91"/>
+<wire x1="63.5" y1="101.6" x2="73.66" y2="101.6" width="0.1524" layer="91"/>
+<wire x1="73.66" y1="101.6" x2="76.2" y2="101.6" width="0.1524" layer="91"/>
 <wire x1="55.88" y1="86.36" x2="71.12" y2="86.36" width="0.1524" layer="91"/>
-<wire x1="55.88" y1="71.12" x2="71.12" y2="71.12" width="0.1524" layer="91"/>
+<wire x1="71.12" y1="86.36" x2="76.2" y2="86.36" width="0.1524" layer="91"/>
+<wire x1="55.88" y1="71.12" x2="73.66" y2="71.12" width="0.1524" layer="91"/>
+<wire x1="73.66" y1="71.12" x2="76.2" y2="71.12" width="0.1524" layer="91"/>
 <wire x1="55.88" y1="48.26" x2="71.12" y2="48.26" width="0.1524" layer="91"/>
+<wire x1="71.12" y1="48.26" x2="76.2" y2="48.26" width="0.1524" layer="91"/>
 <wire x1="55.88" y1="25.4" x2="71.12" y2="25.4" width="0.1524" layer="91"/>
 <pinref part="C1" gate="G$1" pin="+"/>
+<wire x1="71.12" y1="25.4" x2="76.2" y2="25.4" width="0.1524" layer="91"/>
 <wire x1="63.5" y1="106.68" x2="63.5" y2="101.6" width="0.1524" layer="91"/>
-</segment>
-</net>
+<pinref part="TP11" gate="A" pin="TP"/>
+<wire x1="50.8" y1="114.3" x2="55.88" y2="114.3" width="0.1524" layer="91"/>
+<wire x1="55.88" y1="114.3" x2="55.88" y2="101.6" width="0.1524" layer="91"/>
+<pinref part="TP12" gate="G$1" pin="TP"/>
+<wire x1="43.18" y1="114.3" x2="50.8" y2="114.3" width="0.1524" layer="91"/>
+<junction x="55.88" y="101.6"/>
+<junction x="63.5" y="101.6"/>
+<pinref part="TP1" gate="A" pin="TP"/>
+<wire x1="76.2" y1="101.6" x2="76.2" y2="104.14" width="0.1524" layer="91"/>
+<pinref part="TP4" gate="A" pin="TP"/>
+<wire x1="76.2" y1="99.06" x2="73.66" y2="99.06" width="0.1524" layer="91"/>
+<wire x1="73.66" y1="99.06" x2="73.66" y2="101.6" width="0.1524" layer="91"/>
+<pinref part="TP2" gate="A" pin="TP"/>
+<wire x1="76.2" y1="86.36" x2="76.2" y2="88.9" width="0.1524" layer="91"/>
+<wire x1="71.12" y1="86.36" x2="71.12" y2="81.28" width="0.1524" layer="91"/>
+<pinref part="TP3" gate="A" pin="TP"/>
+<wire x1="71.12" y1="81.28" x2="76.2" y2="81.28" width="0.1524" layer="91"/>
+<pinref part="TP5" gate="A" pin="TP"/>
+<wire x1="73.66" y1="71.12" x2="73.66" y2="63.5" width="0.1524" layer="91"/>
+<pinref part="TP6" gate="A" pin="TP"/>
+<wire x1="73.66" y1="63.5" x2="76.2" y2="63.5" width="0.1524" layer="91"/>
+<pinref part="TP7" gate="A" pin="TP"/>
+<wire x1="71.12" y1="48.26" x2="71.12" y2="40.64" width="0.1524" layer="91"/>
+<pinref part="TP8" gate="A" pin="TP"/>
+<wire x1="71.12" y1="40.64" x2="76.2" y2="40.64" width="0.1524" layer="91"/>
+<pinref part="TP9" gate="A" pin="TP"/>
+<wire x1="76.2" y1="25.4" x2="76.2" y2="27.94" width="0.1524" layer="91"/>
+<pinref part="TP10" gate="A" pin="TP"/>
+<wire x1="76.2" y1="20.32" x2="71.12" y2="20.32" width="0.1524" layer="91"/>
+<wire x1="71.12" y1="20.32" x2="71.12" y2="25.4" width="0.1524" layer="91"/>
+<junction x="73.66" y="101.6"/>
+<junction x="71.12" y="86.36"/>
+<junction x="73.66" y="71.12"/>
+<junction x="71.12" y="48.26"/>
+<junction x="55.88" y="48.26"/>
+<junction x="55.88" y="60.96"/>
+<junction x="55.88" y="71.12"/>
+<junction x="55.88" y="81.28"/>
+<junction x="55.88" y="86.36"/>
+<junction x="55.88" y="38.1"/>
+<junction x="71.12" y="25.4"/>
+<junction x="55.88" y="25.4"/>
+</segment>
+</net>
